File: electronics/PSU/pcb/psu.kicad_pcb (KiCad board)
At the start: 2 copper layers, 73 x 80 mm, 132 parts, among them J1 Conn_01x02_Socket, J2 Conn_01x02_Socket, J3 Conn_01x02_Socket, J4 Conn_01x02_Socket, J5 Conn_01x02_Socket, J6 Conn_01x02_Socket, J7 Conn_01x02_Socket, J8 Conn_01x02_Socket, U1 ADPL16000B, U2 LTC3260xDE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

Commit message: update pcb signature
Parts:
- added G***: LOGO, Symbol:nami_logo_4.5mm, F.Cu at (-2.00, 8.00)
Other:
- board text added: "KN NaMi Nanopositioner PSU v.1.0 Jędrzej Soszyński"
- board text removed: "KN-NAMI"
- board text removed: "Nanopositioner PSU v.1.0"
